Commit message: First setup draft

File: inverse_bringup/urdf/prisma.urdf.xacro (robot description, xacro)
@@ -4,5 +4,5 @@
   <link name="world"/>
   <joint name="world_joint" type="fixed">
-    <origin rpy="0 0 0" xyz="0 0 0.2"/>
+    <origin rpy="${pi} 0 0" xyz="0 0 0.2"/>
     <parent link="world"/>
     <child link="table"/>
@@ -90,4 +90,10 @@
                       >
   </xacro:franka_robot>
+  <link name="franka1_tcp"/>
+  <joint name="franka1_flange_to_tcp" type="fixed">
+    <parent link="franka1_fr3_hand_tcp"/>
+    <child link="franka1_tcp"/>
+    <origin xyz="0.0 0.0 0.126" rpy="0 0 0"/>
+  </joint>
   <!-- Dimensions taken from technical drawing of Franka plate and custom designed plate, do not touch -->
   <joint name="table_to_franka2" type="fixed">
@@ -123,4 +129,10 @@
                       >
   </xacro:franka_robot>
+  <link name="franka2_tcp"/>
+  <joint name="franka2_flange_to_tcp" type="fixed">
+    <parent link="franka2_fr3_hand_tcp"/>
+    <child link="franka2_tcp"/>
+    <origin xyz="0.0 0.0 0.11" rpy="0 0 0"/>
+  </joint>
   <!-- Dimensions taken from technical drawing of Franka plate and custom designed plate, do not touch -->
   <joint name="table_to_franka1" type="fixed">

Commit message: WIP

File: inverse_bringup/urdf/prisma.urdf.xacro (robot description, xacro)
@@ -4,5 +4,5 @@
   <link name="world"/>
   <joint name="world_joint" type="fixed">
-    <origin rpy="${pi} 0 0" xyz="0 0 0.2"/>
+    <origin rpy="0 0 0" xyz="0 0 0.2"/>
     <parent link="world"/>
     <child link="table"/>
