Commit message: Add robotiq gripper open test

File: easy_ur_control/urdf/ur_wrapper.xacro (robot description, xacro)
@@ -3,4 +3,5 @@
     <!-- Include the standard UR robot -->
     <xacro:include filename="$(find ur_description)/urdf/ur.urdf.xacro" />
+    <xacro:include filename="$(find robotiq_description)/urdf/robotiq_2f_85_macro.urdf.xacro" />
     <!-- Include your custom gripper and add the joint to connect to it, then go to the
     ur_controllers.yaml and change the ee link in the controller parameters -->
@@ -9,5 +10,23 @@
         <parent link="tool0" />
         <child link="gripper_link" />
+        <origin xyz="0 0 0" rpy="0 0 0" /> -->
+    <xacro:include filename="$(find rokubimini_description)/urdf/BFT_SENS_SER_M8.urdf.xacro" />
+    <xacro:arg name="prefix" default="ft_sensor0" />
+    <!-- Forwarded from launch files; keeps Robotiq in fake mode for sim-only runs. -->
+    <xacro:arg name="use_fake_hardware" default="false" />
+    <xacro:BFT_SENS_SER_M8 prefix="$(arg prefix)" />
+    <joint name="tool0_to_bota" type="fixed">
+        <parent link="tool0" />
+        <child link="$(arg prefix)_mounting" />
+        <origin xyz="0 0 0" rpy="0 0 -${pi/2}" />
+    </joint>
+    <!-- <joint name="robotiq_2f_85_joint" type="fixed">
+      <parent link="tool0" />
+      <origin xyz="0 0 0" rpy="0 0 0" />
+    </joint> -->
+    <!-- Enable ros2_control interfaces for Robotiq and share fake-hardware mode. -->
+    <xacro:robotiq_gripper name="RobotiqGripper" prefix="" parent="ft_sensor0_wrench"
+        include_ros2_control="true" use_fake_hardware="$(arg use_fake_hardware)">
         <origin xyz="0 0 0" rpy="0 0 0" />
-    </joint> -->
+    </xacro:robotiq_gripper>
 </robot>

Commit message: added smpl perception

File: easy_ur_control/urdf/ur_wrapper.xacro (robot description, xacro)
@@ -3,5 +3,5 @@
     <!-- Include the standard UR robot -->
     <xacro:include filename="$(find ur_description)/urdf/ur.urdf.xacro" />
-    <xacro:include filename="$(find robotiq_description)/urdf/robotiq_2f_85_macro.urdf.xacro" />
+    <xacro:include filename="$(find robotiq_description)/urdf/robotiq_2f_140_macro.urdf.xacro" />
     <!-- Include your custom gripper and add the joint to connect to it, then go to the
     ur_controllers.yaml and change the ee link in the controller parameters -->
@@ -21,8 +21,4 @@
         <origin xyz="0 0 0" rpy="0 0 -${pi/2}" />
     </joint>
-    <!-- <joint name="robotiq_2f_85_joint" type="fixed">
-      <parent link="tool0" />
-      <origin xyz="0 0 0" rpy="0 0 0" />
-    </joint> -->
     <!-- Enable ros2_control interfaces for Robotiq and share fake-hardware mode. -->
     <xacro:robotiq_gripper name="RobotiqGripper" prefix="" parent="ft_sensor0_wrench"
@@ -30,3 +26,10 @@
         <origin xyz="0 0 0" rpy="0 0 0" />
     </xacro:robotiq_gripper>
+    <link name="target_link">
+    </link>
+    <joint name="final_joint" type="fixed">
+        <parent link="ft_sensor0_wrench" />
+        <origin xyz="0 0 0.24" rpy="0 0 0" />
+        <child link="target_link" />
+    </joint>
 </robot>

Commit message: Fixed Robotiq gripper with ros2 control and added test

File: easy_ur_control/urdf/ur_wrapper.xacro (robot description, xacro)
@@ -6,24 +6,17 @@
     <xacro:arg name="com_port" default="/dev/ttyUSB0" />
     <xacro:include filename="$(find robotiq_description)/urdf/robotiq_2f_140_macro.urdf.xacro" />
-    <!-- Include your custom gripper and add the joint to connect to it, then go to the
-    ur_controllers.yaml and change the ee link in the controller parameters -->
-    <!-- <xacro:include filename="$(find gripper_description)/urdf/ur_gripper.xacro" /> -->
-    <!-- <joint name="example_gripper_joint" type="fixed">
-        <parent link="tool0" />
-        <child link="gripper_link" />
-        <origin xyz="0 0 0" rpy="0 0 0" /> -->
-    <xacro:include filename="$(find rokubimini_description)/urdf/BFT_SENS_SER_M8.urdf.xacro" />
-    <xacro:arg name="prefix" default="ft_sensor0" />
-    <!-- Forwarded from launch files; keeps Robotiq in fake mode for sim-only runs. -->
     <xacro:arg name="use_fake_hardware" default="false" />
-    <xacro:BFT_SENS_SER_M8 prefix="$(arg prefix)" />
-    <joint name="tool0_to_bota" type="fixed">
-        <parent link="tool0" />
-        <child link="$(arg prefix)_mounting" />
-        <origin xyz="0 0 0" rpy="0 0 -${pi/2}" />
-    </joint>
-    <!-- Enable ros2_control interfaces for Robotiq and share fake-hardware mode. -->
-    <xacro:robotiq_gripper name="RobotiqGripper" prefix="" parent="ft_sensor0_wrench"
-        include_ros2_control="true" use_fake_hardware="$(arg use_fake_hardware)" >
+    <xacro:include filename="$(find robotiq_description)/urdf/ur_to_robotiq_adapter.urdf.xacro" />
+    <xacro:ur_to_robotiq
+        prefix=""
+        parent="tool0"
+        child="robotiq_coupling"
+        rotation="${pi/2}" />
+    <xacro:robotiq_gripper
+        prefix=""
+        parent="robotiq_coupling"
+        name="RobotiqGripper"
+        include_ros2_control="true"
+        use_fake_hardware="$(arg use_fake_hardware)">
         <origin xyz="0 0 0" rpy="0 0 0" />
     </xacro:robotiq_gripper>
@@ -31,6 +24,6 @@
     </link>
     <joint name="final_joint" type="fixed">
-        <parent link="ft_sensor0_wrench" />
-        <origin xyz="0 0 0.24" rpy="0 0 0" />
+        <parent link="robotiq_140_base_link" />
+        <origin xyz="0 0.0 0.2" rpy="0 0 0" />
         <child link="target_link" />
     </joint>
