Commit message: Add Robotiq FT 300

File: easy_ur_control/urdf/ur_wrapper.xacro (robot description, xacro)
@@ -8,7 +8,32 @@
     <xacro:arg name="use_fake_hardware" default="false" />
     <xacro:include filename="$(find robotiq_description)/urdf/ur_to_robotiq_adapter.urdf.xacro" />
+    <!--Include the two macros from robotiq_ft_sensor_description: mechanical-->
+    <xacro:include filename="$(find robotiq_ft_sensor_description)/urdf/robotiq_ft300.urdf.xacro" />
+    <!-- The fts_ros2_control tells the controller manager to load the RobotiqFTSensorHardware plugin and expode force.x/y/-->
+    <xacro:include filename="$(find robotiq_ft_sensor_description)/urdf/robotiq_fts.ros2_control.xacro" />
+    <!-- Robotiq FT 300 force-torque sensor mounted on the flange tool0 with same orientation as tool0-->
+    <xacro:robotiq_ft300 parent="tool0" tf_prefix="">
+        <origin xyz="0 0 0" rpy="0 0 0" />
+    </xacro:robotiq_ft300>
+    <!-- In fake mode the plugin does not open the serial port and reads zeros -->
+    <xacro:robotiq_fts_ros2_control
+        name=""
+        tf_prefix=""
+        use_fake_mode="$(arg use_fake_hardware)"
+        max_retries="100"
+        read_rate="10"
+        ftdi_id="" />
+    <!-- Tool-side face of the sensor (41.5 mm from tool0), same orientation as tool0:
+         robotiq_ft_frame_id is tool0 rotated by +pi/2 around z, so undo that rotation -->
+    <link name="ft300_tool_flange" />
+    <joint name="ft300_tool_flange_joint" type="fixed">
+        <parent link="robotiq_ft_frame_id" />
+        <origin xyz="0 0 0" rpy="0 0 ${-pi/2}" />
+        <child link="ft300_tool_flange" />
+    </joint>
+    <!-- Change from tool0 to ft300_tool_flange -->
     <xacro:ur_to_robotiq
         prefix=""
-        parent="tool0"
+        parent="ft300_tool_flange"
         child="robotiq_coupling"
         rotation="${pi/2}" />

Commit message: Add connector STL and URDF update

File: easy_ur_control/urdf/ur_wrapper.xacro (robot description, xacro)
@@ -14,6 +14,35 @@
     <!-- The fts_ros2_control tells the controller manager to load the RobotiqFTSensorHardware plugin and expode force.x/y/-->
     <xacro:include filename="$(find robotiq_ft_sensor_description)/urdf/robotiq_fts.ros2_control.xacro" />
-    <!-- Robotiq FT 300 force-torque sensor mounted on the flange tool0 with same orientation as tool0-->
-    <xacro:robotiq_ft300 parent="tool0" tf_prefix="">
+    <!-- Connector plate between the UR flange and the FT sensor (mesh in mm, plate axis along mesh +y, 10 mm thick) -->
+    <link name="connector_link">
+        <visual>
+            <origin xyz="0 0 -0.004" rpy="${pi/2} 0 0" />
+            <geometry>
+                <mesh filename="package://easy_ur_control/meshes/connector.stl" scale="0.001 0.001 0.001" />
+            </geometry>
+            <material name="connector_grey">
+                <color rgba="0.75 0.75 0.75 1.0" />
+            </material>
+        </visual>
+        <collision>
+            <origin xyz="0 0 -0.004" rpy="${pi/2} 0 0" />
+            <geometry>
+                <mesh filename="package://easy_ur_control/meshes/connector.stl" scale="0.001 0.001 0.001" />
+            </geometry>
+        </collision>
+    </link>
+    <joint name="tool0_to_connector" type="fixed">
+        <parent link="tool0" />
+        <child link="connector_link" />
+        <origin xyz="0 0 0.01" rpy="0 ${pi} ${pi/2}" />
+    </joint>
+    <link name="connector_tool_side" />
+    <joint name="connector_to_tool_side" type="fixed">
+        <parent link="connector_link" />
+        <child link="connector_tool_side" />
+        <origin xyz="0 0 0.000" rpy="${pi} 0 0" />
+    </joint>
+    <!-- Robotiq FT 300 force-torque sensor mounted on the connector plate with same orientation as tool0-->
+    <xacro:robotiq_ft300 parent="connector_tool_side" tf_prefix="">
         <origin xyz="0 0 0" rpy="0 0 0" />
     </xacro:robotiq_ft300>

Commit message: Integrate Realsense in URDF

File: easy_ur_control/urdf/ur_wrapper.xacro (robot description, xacro)
@@ -85,3 +85,8 @@
         <child link="target_link" />
     </joint>
+    <!-- D435if uses the D435i housing and frame model. -->
+    <xacro:include filename="$(find realsense2_description)/urdf/_d435i.urdf.xacro" />
+    <xacro:sensor_d435i parent="connector_tool_side" name="camera">
+        <origin xyz="0.085 0 0.01" rpy="${pi} -${pi/2} 0" />
+    </xacro:sensor_d435i>
 </robot>

Commit message: Add update finger tips to URDF

File: easy_ur_control/urdf/ur_wrapper.xacro (robot description, xacro)
@@ -78,9 +78,41 @@
         <origin xyz="0 0 0" rpy="0 0 0" />
     </xacro:robotiq_gripper>
+    <!-- Finger tips -->
+    <link name="left_finger_tip">
+        <visual>
+            <!-- Tip dimensions: x = 8 mm, y = 100 - 32.5 mm, z = 4 mm. -->
+            <!-- Apply offset of y/2 -->
+            <origin xyz="0.0 0.03375 0.0015" />
+            <geometry>
+                <box size="0.008 0.0675 0.004" />
+            </geometry>
+        </visual>
+    </link>
+    <joint name="left_finger_tip_joint" type="fixed">
+        <parent link="left_inner_finger_pad" />
+        <origin xyz="0.0 0.0 0.0" rpy="0.0 0.0 0.0" />
+        <child link="left_finger_tip" />
+    </joint>
+    <link name="right_finger_tip">
+        <visual>
+            <!-- Tip dimensions: x = 8 mm, y = 100 - 32.5 mm, z = 4 mm. -->
+            <!-- Apply offset of y/2 -->
+            <origin xyz="0.0 0.03375 0.0015" />
+            <geometry>
+                <box size="0.008 0.0675 0.004" />
+            </geometry>
+        </visual>
+    </link>
+    <joint name="right_finger_tip_joint" type="fixed">
+        <parent link="right_inner_finger_pad" />
+        <origin xyz="0.0 0.0 0.0" rpy="0.0 0.0 0.0" />
+        <child link="right_finger_tip" />
+    </joint>
+    <!-- Controlled reference frame -->
     <link name="target_link">
     </link>
     <joint name="final_joint" type="fixed">
         <parent link="robotiq_140_base_link" />
-        <origin xyz="0 0.0 0.2" rpy="0 0 0" />
+        <origin xyz="0 0.0 0.2675" rpy="0 0 0" />
         <child link="target_link" />
     </joint>

Commit message: Register aruco marker frame

File: easy_ur_control/urdf/ur_wrapper.xacro (robot description, xacro)
@@ -122,3 +122,11 @@
         <origin xyz="0.085 0 0.01" rpy="${pi} -${pi/2} 0" />
     </xacro:sensor_d435i>
+    <!-- Aruco frame -->
+    <link name="aruco_link">
+    </link>
+    <joint name="aruco_joint" type="fixed">
+        <parent link="base_link" />
+        <origin xyz="0 0.91 0.04" rpy="0 0 -${pi/2}" />
+        <child link="aruco_link" />
+    </joint>
 </robot>

Commit message: Update RS placement in urdf

File: easy_ur_control/urdf/ur_wrapper.xacro (robot description, xacro)
@@ -120,5 +120,5 @@
     <xacro:include filename="$(find realsense2_description)/urdf/_d435i.urdf.xacro" />
     <xacro:sensor_d435i parent="connector_tool_side" name="camera">
-        <origin xyz="0.085 0 0.01" rpy="${pi} -${pi/2} 0" />
+        <origin xyz="0.077 0 0.01" rpy="${pi} -${pi/2} ${pi}" />
     </xacro:sensor_d435i>
     <!-- Aruco frame -->
